File: Back/Back.kicad_pcb (KiCad board)
At the start: 2 copper layers, 338.8 x 124.7 mm, 8 parts

Commit message: Update top offset
Parts:
- moved H7 12.4 mm to (277.5, 217.9)
- moved H2 4.35 mm to (161.6, 218.3)
- moved H5 1.55 mm to (52.9, 107.5)
- moved H1 1.37 mm to (277.5, 107.5)
- moved H3 1.37 mm to (383.9, 107.5)
- moved H8 1.37 mm to (161.6, 107.5)
- moved H6 0.16 mm to (52.9, 210.2)
- moved H4 0.13 mm to (383.9, 210.2)
Connections:
- H1 pad 1: unconnected-(H1-Pad1) -> GND
- H2 pad 1: unconnected-(H2-Pad1) -> GND
- H3 pad 1: unconnected-(H3-Pad1) -> GND
- H4 pad 1: unconnected-(H4-Pad1) -> GND
- H5 pad 1: unconnected-(H5-Pad1) -> GND
- H6 pad 1: unconnected-(H6-Pad1) -> GND
- H7 pad 1: unconnected-(H7-Pad1) -> GND
- H8 pad 1: unconnected-(H8-Pad1) -> GND
Routing:
- added copper zone on B.Cu, net GND
- added copper zone on F.Cu, net GND
Other:
- board size 338.8 x 124.7 mm -> 338.8 x 126.5 mm
- board text added: "(This side goes down)"
- board text added: "FRONT TOWARD ENEMY"
