File: Plate/Plate.kicad_pcb (KiCad board)
At the start: 2 copper layers, 338.8 x 124.7 mm, 8 parts

Commit message: Update top offset
Parts:
- moved H7 12.4 mm to (277.5, 217.9)
- moved H2 4.35 mm to (161.6, 218.3)
- moved H5 1.55 mm to (52.9, 107.5)
- moved H1 1.37 mm to (277.5, 107.5)
- moved H3 1.37 mm to (383.9, 107.5)
- moved H8 1.37 mm to (161.6, 107.5)
- moved H6 0.16 mm to (52.9, 210.2)
- moved H4 0.13 mm to (383.9, 210.2)
Connections:
- H1 pad 1: unconnected-(H1-Pad1) -> GND
- H2 pad 1: unconnected-(H2-Pad1) -> GND
- H3 pad 1: unconnected-(H3-Pad1) -> GND
- H4 pad 1: unconnected-(H4-Pad1) -> GND
- H5 pad 1: unconnected-(H5-Pad1) -> GND
- H6 pad 1: unconnected-(H6-Pad1) -> GND
- H7 pad 1: unconnected-(H7-Pad1) -> GND
- H8 pad 1: unconnected-(H8-Pad1) -> GND
Routing:
- added copper zone on B.Cu, net GND
- added copper zone on F.Cu, net GND
Other:
- board size 338.8 x 124.7 mm -> 338.8 x 126.5 mm

Commit message: Updated stuff
Other:
- board text added: "JLCJLCJLCJLC"
Changed lines of the file:
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@@
   (gr_line (start 121.801527 135.533669) (end 121.801527 147.533669) (layer "Edge.Cuts") (width 0.2))
   (gr_curve (pts (xy 162.539916 195.976597) (xy 162.502257 195.963749) (xy 162.463865 195.953161) (xy 162.424944 195.944888)) (layer "Edge.Cuts") (width 0.2))
+  (gr_text "JLCJLCJLCJLC" (at 323.05625 210.34375) (layer "B.SilkS")
+    (effects (font (size 1 1) (thickness 0.2)) (justify mirror))
+  )
   (zone (net 1) (net_name "GND") (layers F&B.Cu) (hatch edge 0.508)
     (connect_pads yes (clearance 0.3))
